Commit message: Added scanse sweep lidar to robot urdf

File: turtlebot3_description/urdf/turtlebot3_waffle.urdf.xacro (robot description, xacro)
@@ -140,11 +140,11 @@
     <parent link="base_link"/>
     <child link="base_scan"/>
-    <origin xyz="-0.064 0 0.122" rpy="0 0 0"/>
+    <origin xyz="-0.064 0 0.122" rpy="0 0 -1.5708"/>
   </joint>
   <link name="base_scan">
     <visual>
-      <origin xyz="0 0 0" rpy="0 0 0"/>
-      <geometry>
-        <mesh filename="package://turtlebot3_description/meshes/sensors/lds.stl" scale="0.001 0.001 0.001"/>
+      <origin xyz="0 -0.02 0" rpy="0 0 -1.5708"/>
+      <geometry>
+        <mesh filename="package://turtlebot3_description/meshes/sensors/sweep_lidar.stl" scale="1 1 1"/>
       </geometry>
       <material name="dark"/>

Commit message: changes config to default LIDAR

File: turtlebot3_description/urdf/turtlebot3_waffle.urdf.xacro (robot description, xacro)
@@ -140,11 +140,11 @@
     <parent link="base_link"/>
     <child link="base_scan"/>
-    <origin xyz="-0.064 0 0.122" rpy="0 0 -1.5708"/>
+    <origin xyz="-0.064 0 0.122" rpy="0 0 0"/>
   </joint>
   <link name="base_scan">
     <visual>
-      <origin xyz="0 -0.02 0" rpy="0 0 -1.5708"/>
-      <geometry>
-        <mesh filename="package://turtlebot3_description/meshes/sensors/sweep_lidar.stl" scale="1 1 1"/>
+      <origin xyz="0 0 0" rpy="0 0 0"/>
+      <geometry>
+        <mesh filename="package://turtlebot3_description/meshes/sensors/lds.stl" scale="0.001 0.001 0.001"/>
       </geometry>
       <material name="dark"/>
